File: Kicad/grove-breakout.kicad_pcb (KiCad board)
At the start: 2 copper layers, 38.1 x 71 mm, 12 parts, among them J1 Conn_01x15_Pin, J10 UEXT, J2 Grove_LIGHT, J3 Grove_POT, J4 Grove_STICK, J5 Grove_I2C, J6 Grove_DHT11, J7 Grove_BUZZER, J8 Grove_RELAY, J9 Grove_BUTTON

Commit message: Sanity
Parts:
- added J5: Grove_I2C, Connector_JST:JST_PH_B4B-PH-K_1x04_P2.00mm_Vertical, F.Cu at (134.1, 104.5)
Routing:
- net I2C_SDA_IO26: track 46.3 -> 58.7 mm
- net I2C_SCL_IO27: track 33.1 -> 40.1 mm
Other:
- board text added: "LED"
- board text added: "MOSI IO23"
- board text added: "RXD IO35"
- board text added: "SDA IO26"
- board text added: "SSEL IO5"
- board text added: "TXD IO22"
- board text removed: "1 3V3 #1"
- board text removed: "3 TXD IO22 #7"
- board text removed: "GND #2 2"
- board text removed: "MOSI IO23 #9 J8 8"
- board text removed: "NO 5V"
- board text removed: "RXD IO35 #5 4"
- board text removed: "SDA IO26 #15 J5 6"
- board text removed: "SSEL IO5 #13 10"
- board text removed: "STICK"

Commit message: top copper
Routing:
- added copper zone on F.Cu, net GND
Changed lines of the file:
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@@
+	(zone
+		(net "GND")
+		(layer "F.Cu")
+		(hatch edge 0.5)
+		(priority 1)
+		(connect_pads
+			(clearance 0.5)
+		)
+		(min_thickness 0.25)
+		(fill yes
+			(thermal_gap 0.5)
+			(thermal_bridge_width 0.5)
+			(island_removal_mode 0)
+		)
+		(polygon
+			(pts
+				(xy 95 79.5) (xy 142 79.5) (xy 140.5 160) (xy 92.5 159.5) (xy 95.5 85)
+			)
+		)
+	)
 	(zone
 		(net "GND")
